Commit message: Hoofdprogrammawerktnuechtgeweldigg

File: src/my_xarm_lite6/my_lite6_description/urdf/robotopstelling.urdf.xacro (robot description, xacro)
@@ -8,5 +8,5 @@
     <link name="Opstelling_Link">
   <visual>
-    <origin xyz="0 0 0" rpy="0 0 -${pi/2}" /> <!-- Verplaats het object naar de juiste plek -->
+    <origin xyz="-0.1 0.03 0" rpy="0 0 -${pi/2}" /> <!-- Verplaats het object naar de juiste plek -->
     <geometry>
       <mesh filename="package://my_lite6_description/meshes/AssmOpstellingV3.STL" scale="1.00 1.00 1.00"/>
@@ -17,5 +17,5 @@
   </visual>
   <collision>
-    <origin xyz="0 0 0" rpy="0 0 -${pi/2}" />		<!-- ${pi/2} -->
+    <origin xyz="-0.1 0.03 0" rpy="0 0 -${pi/2}" />		<!-- ${pi/2} -->
     <geometry>
       <mesh filename="package://my_lite6_description/meshes/AssmOpstellingV3.STL" scale="1.00 1.00 1.00"/>

File: src/xarm_ros/xarm_description/urdf/gripper/lite_gripper.urdf.xacro (robot description, xacro)
@@ -24,6 +24,6 @@
       <xacro:common_link_collision
         mesh_filename="gripper/lite/collision/gripper_lite"
-        origin_xyz="0 0 0"
-        origin_rpy="0 0 0" />
+        origin_xyz="-0.095 0.0075 0.0811"
+        origin_rpy="${pi} 0 0" />
     </link>
     <link name="${prefix}link_tcp" />
